File: CANdlestick.v2/particle-can-v2.0.brd (EAGLE design)
At the start: 29 x 32.3 mm, 13 parts, among them IC1 LM2940, IC2 TJA1049, J1 OBDII

Commit message: Version 2 of the PCB has optimized components and GPS
Parts:
- C3: value 24u -> 22u
- C4: value 0.1u -> 3.3u
- CORE: device Particle:PHOTON_STACKABLE_EXTERNAL -> MuniRent:PHOTON_STACKABLE_EXTERNAL
- D1: device BUG:SOT23 -> MuniRent:SOT23
- GPS: device SparkFun-Connectors:JST-6-SMD-HOR-1.0MM -> MuniRent:JST-6-SMD-HOR-1.0MM
- IC1: device BUG:SOT223 -> MuniRent:SOT223
- IC2: device BUG:SO8 -> MuniRent:SO8
- J1: device BUG:OBDII-STRAIGHT -> MuniRent:OBDII-STRAIGHT
