File: CANdlestick.v2/particle-can-v2.1.sch (EAGLE design)
At the start: 22 parts, among them IC1 NCP1117, IC2 TJA1049, J1 OBDII

Commit message: Revision 2.1 and 3.1
Parts:
- removed C2: 10u, rcl:C-EUC0805
- removed C4: DNP, rcl:C-EUC0805
- removed C6: 0.1u, rcl:C-EUC0805
- removed C7: 1u, rcl:C-EUC0805
- removed D3: RS1J, BUG:DIODESMA
- removed ELECTRON: ELECTRON_WITH_EXTERNAL_HEADERS, MuniRent:ELECTRON_WITH_EXTERNAL_HEADERS
- removed SDCARD: USD-SOCKETMOLEX, MuniRent:USD-SOCKETMOLEX
- removed STANDOFF1, STANDOFF2: STAND-OFF, SparkFun-Electromechanical:STAND-OFF
- removed TP1: CANH, SparkFun-Passives:TEST-POINT3
- removed TP2: CANL, SparkFun-Passives:TEST-POINT3
- removed TP3: 12V, SparkFun-Passives:TEST-POINT3
- removed TP5: 3.3V, SparkFun-Passives:TEST-POINT3
- added CORE: PHOTONWITH_EXTERNAL_HEADERS, MuniRent:PHOTONWITH_EXTERNAL_HEADERS
- added R1: 62k, rcl:R-US_R0805
- added R2: 10k, rcl:R-US_R0805
- added U$1, U$5: LOGOSMALL, MuniRent:LOGOSMALL
- GPS: value JST -> JST_VERTICALHORIZONTAL; device MuniRent:JST -> MuniRent:JST_VERTICALHORIZONTAL; PARTNO BM06B-SRSS-TB -> SM06B-SRSS-TB
- IC1: value NCP1117 -> LM2940; device MuniRent:NCP1117 -> MuniRent:LM2940; PARTNO NCP1117LPST50T3G -> LM2940IMP-5.0/NOPB
- J1: device MuniRent:M08X2-OBDII-COMTECH -> MuniRent:M08X2STRAIGHT
Connections:
- removed net N$1: ELECTRON.B5
- removed net N$17: ELECTRON.B3
- removed net N$18: ELECTRON.A1
- removed net N$21: ELECTRON.B0
- removed net N$22: ELECTRON.C0
- removed net N$27: ELECTRON.C4
- removed net N$28: ELECTRON.C5
- removed net N$29: ELECTRON.C3
- removed net N$31: C2.1, D3.C, IC1.IN
- removed net N$7: ELECTRON.B4
- removed net SD_CS: ELECTRON.A2, SDCARD.CS
- removed net SPI_MISO: ELECTRON.A4, SDCARD.DO
- removed net SPI_MOSI: ELECTRON.A5, SDCARD.DI
- removed net SPI_SCK: ELECTRON.A3, SDCARD.SCK
- new net VBAT: CORE.A1, R1.1, R2.2
- net +12V: now also IC1.IN, R1.2; no longer D3.A, TP3.1
- net 3.3V: now also CORE.3V3; no longer C6.1, C7.1, ELECTRON.3V3, SDCARD.VCC, TP5.1
- net 5V: now also CORE.VIN; no longer C4.1, ELECTRON.VIN
- net CANA_EN: now also CORE.D0; no longer ELECTRON.D0
- net CANA_RX: now also CORE.D2; no longer ELECTRON.D2
- net CANA_TX: now also CORE.D1; no longer ELECTRON.D1
- net GND: now also CORE.GND@2, R2.1; no longer C2.2, C4.2, C6.2, C7.2, ELECTRON.GND@2, SDCARD.CD1, SDCARD.CD2, SDCARD.GND, SDCARD.SHIELD@1, SDCARD.SHIELD@3
- net GPS_EN: now also CORE.A0; no longer ELECTRON.A0
- net GPS_RX: now also CORE.TX; no longer ELECTRON.TX
- net GPS_TX: now also CORE.RX; no longer ELECTRON.RX
- net HSPD_HI: now also D1.C1; no longer D1.C2, TP1.1
- net HSPD_LO: now also D1.C2; no longer D1.C1, TP2.1
- net N$10: now also CORE.!RST; no longer ELECTRON.!RST
- net N$11: now also CORE.VBAT; no longer ELECTRON.VBAT
- net N$12: now also CORE.D7; no longer ELECTRON.D7
- net N$13: now also CORE.D6; no longer ELECTRON.D6
- net N$14: now also CORE.D5; no longer ELECTRON.D5
- net N$15: now also CORE.D4; no longer ELECTRON.D4
- net N$16: now also CORE.D3; no longer ELECTRON.D3
- net N$19: now also CORE.A2; no longer ELECTRON.B2
- net N$20: now also CORE.A3; no longer ELECTRON.B1
- net N$23: now also CORE.A4; no longer ELECTRON.C1
- net N$24: now also CORE.A5; no longer ELECTRON.C2
- net N$25: now also CORE.DAC; no longer ELECTRON.DAC
- net N$26: now also CORE.WKP; no longer ELECTRON.WKP
Other:
- note added: "Battery voltage"
- note removed: "Micro SD Card"
- moved on the sheet: C1, D2
