File: CANdlestick.v2/particle-can-v2.3.brd (EAGLE design)
At the start: 31.8 x 37.8 mm, 21 parts, among them IC1 RT8258, IC2 TJA1049, J1 OBDII

Commit message: Add BOM and Gerber files for Rev 2.3
Parts:
- R4: value 91k -> 17.4k
- moved C2 1.09 mm to (17.0, 28.3)
Routing:
- net N$1: track 13.9 -> 14.8 mm
- net GND: vias 8 -> 17
Other:
- board text added: "VBAT"
- board text removed: "12V"
