File: CANdlestick.v2/particle-can-v2.3.sch (EAGLE design)
At the start: 19 parts, among them IC1 RT8258, IC2 TJA1049, J1 OBDII

Commit message: Add BOM and Gerber files for Rev 2.3
Parts:
- C1: PARTNO (none) -> GRM31CR61E106KA12L
- C2: PARTNO (none) -> C0402C103K5RACTU
- C3: PARTNO (none) -> GRM31CR61C226ME15L
- C5: PARTNO 08055C104KAT2A -> GRM155R71C104KA88D
- D3: PARTNO (none) -> B230A-13-F
- IC1: PARTNO (none) -> RT8258GJ6
- L1: PARTNO (none) -> NR8040T150M
- R1: PARTNO ERJ-6ENF6202V -> ERJ-2RKF6202X
- R2: PARTNO ERJ-6ENF1002V -> ERJ-2RKF1002X
- R3: PARTNO ERJ-6ENF6202V -> ERJ-2RKF9102X
- R4: value 91k -> 17.4k; PARTNO ERJ-6ENF6202V -> ERJ-2RKF1742X
