File: CANdlestick.v3/particle-can-v3.1.sch (EAGLE design)
At the start: 22 parts, among them IC1 NCP1117, IC2 TJA1049, J1 OBDII

Commit message: Revision 2.1 and 3.1
Parts:
- added D4: BAT54S, MuniRent:BAT54S
- added R1: 62k, rcl:R-US_R0805
- added R2: 10k, rcl:R-US_R0805
- added U$1: LOGO, MuniRent:LOGO
- IC1: value NCP1117 -> NCP1117CORRECT; device MuniRent:NCP1117 -> MuniRent:NCP1117CORRECT
- SDCARD: value USD-SOCKETMOLEX -> USD-SOCKETMOLEX-CORRECT; device MuniRent:USD-SOCKETMOLEX -> MuniRent:USD-SOCKETMOLEX-CORRECT
- STANDOFF1, STANDOFF2, TP1, TP2, TP3, TP5: BOM (none) -> EXCLUDE
Connections:
- removed net N$18: ELECTRON.A1
- removed net N$25: ELECTRON.DAC
- new net SD_DETECT: ELECTRON.DAC, SDCARD.CD2
- new net VBAT: D4.COM, ELECTRON.A1, R1.1, R2.2
- net +12V: now also R1.2
- net 3.3V: now also D4.C1
- net GND: now also D4.A2, R2.1; no longer SDCARD.CD2
Other:
- note added: "Battery voltage"
- moved on the sheet: GPS
