File: Carloop2.v3/Carloop2-v3.1.brd (EAGLE design)
At the start: 57.8 x 40.6 mm, 32 parts, among them IC1 RT8258, IC2 AZ1117E, IC3 TJA1049, IC4 MCP2517FD, J1 OBDII, Q1 40MHz

Commit message: First prototype of Carloop 2
Parts:
- C11, C12: value 10u -> 22uF
- C2: value 10n -> 10nF; device rcl:C0402 -> rcl:C0603
- C3: value 22u -> 22uF
- C4, C5: device rcl:C0805 -> rcl:C0603
- C6, C7, C8: value 0.1u -> 0.1uF; device rcl:C0402 -> rcl:C0603
- R1, R2, R3, R4: device rcl:R0402 -> rcl:R0603
- moved R4 0.36 mm to (42.9, 21.3)
- moved R3 0.28 mm to (45.2, 21.3)
- moved C8 0.28 mm to (13.7, 17.0)
- moved C2 0.28 mm to (47.2, 17.0)
- moved R1 0.25 mm to (34.3, 39.0)
- moved C7 0.18 mm to (17.3, 17.0)
- renumbered U$1 to IC5
Routing:
- net 3.3V: track 60.1 -> 59.3 mm
- net +12V: track 101.8 -> 102.5 mm
Other:
- board text added: "12V"
- board text added: "CANH"
- board text added: "CANL"
- board text added: "GND"
