File: Carloop2.v3/Carloop2-v3.1.sch (EAGLE design)
At the start: 30 parts, among them IC1 RT8258, IC2 AZ1117E, IC3 TJA1049, IC4 MCP2517FD, J1 OBDII, Q1 40MHz

Commit message: First prototype of Carloop 2
Parts:
- C1: PARTNO GRM31CR61E106KA12L -> C3216X7R1E106K160AB
- C11, C12: value 10u -> 22uF; PARTNO GRM31CR61C226ME15L -> CL31X226KAHN3NE
- C2: value 10n -> 10nF; device rcl:C-EUC0402 -> rcl:C-EUC0603; PARTNO C0402C103K5RACTU -> CGA3E2X8R1H103K080AA
- C3: value 22u -> 22uF; PARTNO GRM31CR61C226ME15L -> CL31X226KAHN3NE
- C4, C5: device rcl:C-EUC0805 -> rcl:C-EUC0603; PARTNO C0805C220J5GACTU -> CC0603KRX7R9BB223
- C6, C8: value 0.1u -> 0.1uF; device rcl:C-EUC0402 -> rcl:C-EUC0603; PARTNO C0402C103K5RACTU -> CC0603JRX7R7BB104
- C7: value 0.1u -> 0.1uF; device rcl:C-EUC0402 -> rcl:C-EUC0603; PARTNO GRM155R71C104KA88D -> CC0603JRX7R7BB104
- D4, D5: PARTNO (none) -> MBRA140T3G
- IC2: PARTNO (none) -> AZ1117EH-3.3TRG1
- IC4: PARTNO (none) -> MCP2517FD-H/SL
- IC5, SJ1, SJ2: BOM (none) -> EXCLUDE
- J2: PARTNO (none) -> OSTTE040104
- Q1: PARTNO ABM3B-16.000MHZ-10-1-U-T -> ECS-400-12-30B-AGM-TR
- R1: device rcl:R-US_R0402 -> rcl:R-US_R0603; PARTNO ERJ-2RKF6202X -> ERA-3AEB623V
- R2: device rcl:R-US_R0402 -> rcl:R-US_R0603; PARTNO ERJ-2RKF1002X -> ERA-3AED103V
- R3: device rcl:R-US_R0402 -> rcl:R-US_R0603; PARTNO ERJ-2RKF9102X -> ERA-3ARB913V
- R4: device rcl:R-US_R0402 -> rcl:R-US_R0603; PARTNO ERJ-2RKF1742X -> ERJ-3EKF1742V
- renumbered U$1 to IC5
